File: hardware/BREAD_Slice.kicad_pcb (KiCad board)
At the start: 2 copper layers, 70 x 100 mm, 33 parts, among them J1 Conn_01x02_Pin, J10 Conn_01x08_Pin, J11 Conn_01x08_Pin, J12 Conn_01x10_Socket, J2 Conn_01x02_Pin, J3 Conn_01x02_Pin, J4 Conn_01x08_Pin, J5 Conn_01x08_Pin, J6 Conn_01x06_Pin, J7 Conn_01x08_Pin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

Commit message: review and revise board and update footprints
Parts:
- A1: footprint kml-custom:Arduino_Nano_Headers -> KMLib_Boards_Modules:Arduino_Nano_Headers
- D2: footprint kml-custom:WS2812-5050-4PIN -> KMLib_IC_SMD:WS2812-5050-4PIN
- G***: footprint kml-custom:FAST-Logo-Medium -> KMLib_Aesthetic:FAST-Logo-Medium
- HS1: footprint kml-custom:Thermal Pad -> KMLib_Mounting:Thermal Pad
- Ref**: footprint kml-custom:OSHW_Logo_8mm -> KMLib_Aesthetic:OSHW_Logo_8mm
- U1: footprint kml-custom:SOIC_05WU-7_DIO-M -> KMLib_IC_SMD:SOIC_05WU-7_DIO
- moved J2 5.07 mm to (169.3, 105.9), turned to 90 degrees
Routing:
- net GND: track 100.4 -> 166.5 mm, vias 19 -> 47
- net /slice_template/~{RESET}: track 18.9 -> 13.9 mm
- net (no net): track 0.00 -> 0.01 mm, vias 464 -> 440
