File: hardware/slice_template.kicad_sch (KiCad schematic)
At the start: 19 parts, among them J12 Conn_01x10_Socket, SW1 SW_DIP_x04, U1 AP63205

Commit message: review and revise board and update footprints
Parts:
- A1: footprint kml-custom:Arduino_Nano_Headers -> KMLib_Boards_Modules:Arduino_Nano_Headers
- D2: footprint kml-custom:WS2812-5050-4PIN -> KMLib_IC_SMD:WS2812-5050-4PIN
- HS1: footprint kml-custom:Thermal Pad -> KMLib_Mounting:Thermal Pad
- U1: footprint kml-custom:SOIC_05WU-7_DIO-M -> KMLib_IC_SMD:SOIC_05WU-7_DIO
Changed lines of the file:
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@@
 			)
 		)
-		(property "Footprint" "kml-custom:Arduino_Nano_Headers"
+		(property "Footprint" "KMLib_Boards_Modules:Arduino_Nano_Headers"
 			(at 237.49 81.28 0)
 			(effects
@@
 			)
 		)
-		(property "Footprint" "kml-custom:SOIC_05WU-7_DIO-M"
+		(property "Footprint" "KMLib_IC_SMD:SOIC_05WU-7_DIO"
 			(at 113.03 93.98 0)
 			(effects
@@
 			)
 		)
-		(property "Footprint" "kml-custom:WS2812-5050-4PIN"
+		(property "Footprint" "KMLib_IC_SMD:WS2812-5050-4PIN"
 			(at 190.5 142.24 0)
 			(effects
@@
 			)
 		)
-		(property "Footprint" "kml-custom:Thermal Pad"
+		(property "Footprint" "KMLib_Mounting:Thermal Pad"
 			(at 68.2752 107.95 0)
 			(effects
