File: hardware/slice_template.kicad_sch (KiCad schematic)
At the start: 19 parts, among them J12 Conn_01x10_Socket, SW1 SW_DIP_x04, U1 AP63205

Commit message: fix(hw): re-point stale library nicknames
These parts exist in KiCad-Master-Lib; the boards referenced libraries that no
longer exist (kml-custom, KML-Custom, and SparkFun libraries that never
contained the part) or names the library has since changed.

KiCad embeds footprint geometry in the .kicad_pcb, so the boards rendered and
fabricated correctly and the rot stayed invisible -- it only surfaces on
update-from-library, or when a generator tries to resolve a nickname.

Nickname/name only. No geometry is changed:

  KMLib_Mounting:Thermal Pad -> KMLib_Mounting:Thermal_Pad
  SparkFun-LED:WS2812-5050-4PIN -> KMLib_IC_SMD:WS2812-5050-4PIN
  kml-custom:AP63205WU-7 -> KMLib_IC_Power:AP63205WU-7_Buck_Regulator
  kml-custom:Arduino_Nano_v3.x -> KMLib_IC_MCU_MPU:Arduino_Nano_v3.x
  kml-custom:SOIC_05WU-7_DIO -> KMLib_IC_SMD:SOIC_05WU-7_DIO
  kml-custom:WS2812B_5050 -> SparkFun-LED:WS2812B_5050

Only references that failed to resolve were touched. Generic parts (<=4 pins)
and KiCad *-rescue libraries are deliberately excluded: fingerprint matching
cannot distinguish a 2-pin resistor from a 2-pin capacitor, so those are being
done by hand.
Parts:
- A1: symbol kml-custom:Arduino_Nano_v3.x -> KMLib_IC_MCU_MPU:Arduino_Nano_v3.x
- D2: symbol kml-custom:WS2812B_5050 -> SparkFun-LED:WS2812B_5050
- HS1: footprint KMLib_Mounting:Thermal Pad -> KMLib_Mounting:Thermal_Pad
- U1: symbol kml-custom:AP63205WU-7 -> KMLib_IC_Power:AP63205WU-7_Buck_Regulator
Changed lines of the file:
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@@
 	)
 	(symbol
-		(lib_id "kml-custom:Arduino_Nano_v3.x")
+		(lib_id "KMLib_IC_MCU_MPU:Arduino_Nano_v3.x")
 		(at 237.49 81.28 0)
 		(unit 1)
@@
 	)
 	(symbol
-		(lib_id "kml-custom:AP63205WU-7")
+		(lib_id "KMLib_IC_Power:AP63205WU-7_Buck_Regulator")
 		(at 113.03 93.98 0)
 		(unit 1)
@@
 	)
 	(symbol
-		(lib_id "kml-custom:WS2812B_5050")
+		(lib_id "SparkFun-LED:WS2812B_5050")
 		(at 173.99 133.35 0)
 		(mirror y)
@@
 			)
 		)
-		(property "Footprint" "KMLib_Mounting:Thermal Pad"
+		(property "Footprint" "KMLib_Mounting:Thermal_Pad"
 			(at 68.2752 107.95 0)
 			(hide yes)
